File: CorneReference.kicad_sch (KiCad schematic)
At the start: 89 parts, among them J1 TYPE-C-31-M-13C, J2 TRS, J3 Conn_01x04, J4 Conn_01x03, SW1 SW_Push, SW10 SW_Push, SW11 SW_Push, SW12 SW_Push, SW13 SW_Push, SW14 SW_Push, SW15 SW_Push, SW16 SW_Push, SW17 SW_Push, SW18 SW_Push, SW19 SW_Push, SW2 SW_Push, SW20 SW_Push, SW21 SW_Push, SW3 SW_Push, SW4 SW_Push, SW5 SW_Push, SW6 SW_Push, SW7 SW_Push, SW8 SW_Push, SW9 SW_Push, U1 RP2040, U2 NCP1117LPST33T3G, U3 TPD4E05U06DQAR, U4 W25Q128JVSIQ, Y1 12MHz 18pF

Commit message: get the Corne reference set up
Parts:
- BT5: renamed from BT1; footprint kbd_local:Breakaway_Tabs -> kbd:Breakaway_Tabs
- BT6: renamed from BT2; footprint kbd_local:Breakaway_Tabs -> kbd:Breakaway_Tabs
- BT7: renamed from BT3; footprint kbd_local:Breakaway_Tabs -> kbd:Breakaway_Tabs
- BT8: renamed from BT4; footprint kbd_local:Breakaway_Tabs -> kbd:Breakaway_Tabs
- EXLED3: renamed from EXLED1; footprint kbd_local:YS-SK6812MINI-E -> kbd:YS-SK6812MINI-E
- EXLED4: renamed from EXLED2; footprint kbd_local:YS-SK6812MINI-E -> kbd:YS-SK6812MINI-E
- EXSW3: renamed from EXSW1; footprint kbd_local:keyswitch_cherrymx_hotswap_1u_rotary_encoder_ec12 -> kbd:keyswitch_cherrymx_hotswap_1u_rotary_encoder_ec12
- EXSW4: renamed from EXSW2; footprint kbd_local:keyswitch_cherrymx_hotswap_1u_rotary_encoder_ec12 -> kbd:keyswitch_cherrymx_hotswap_1u_rotary_encoder_ec12
- J7: renamed from J1; footprint kbd_local:TYPE-C-31-M-13C -> kbd:TYPE-C-31-M-13C
- J8: renamed from J2; footprint kbd_local:PJ-398A-5A_PJ-399B-6A -> kbd:PJ-398A-5A_PJ-399B-6A
- J9: renamed from J3; footprint kbd_local:OLED -> kbd:OLED
- LED34: renamed from LED19; footprint kbd_local:YS-SK6812MINI-E -> kbd:YS-SK6812MINI-E
- LED35: renamed from LED20; footprint kbd_local:YS-SK6812MINI-E -> kbd:YS-SK6812MINI-E
- LED36: renamed from LED21; footprint kbd_local:YS-SK6812MINI-E -> kbd:YS-SK6812MINI-E
- LED37: renamed from LED18; footprint kbd_local:YS-SK6812MINI-E -> kbd:YS-SK6812MINI-E
- LED38: renamed from LED17; footprint kbd_local:YS-SK6812MINI-E -> kbd:YS-SK6812MINI-E
- LED39: renamed from LED16; footprint kbd_local:YS-SK6812MINI-E -> kbd:YS-SK6812MINI-E
- LED40: renamed from LED13; footprint kbd_local:YS-SK6812MINI-E -> kbd:YS-SK6812MINI-E
- LED41: renamed from LED14; footprint kbd_local:YS-SK6812MINI-E -> kbd:YS-SK6812MINI-E
- LED42: renamed from LED15; footprint kbd_local:YS-SK6812MINI-E -> kbd:YS-SK6812MINI-E
- LED43: renamed from LED12; footprint kbd_local:YS-SK6812MINI-E -> kbd:YS-SK6812MINI-E
- LED44: renamed from LED11; footprint kbd_local:YS-SK6812MINI-E -> kbd:YS-SK6812MINI-E
- LED45: renamed from LED10; footprint kbd_local:YS-SK6812MINI-E -> kbd:YS-SK6812MINI-E
- LED46: renamed from LED9; footprint kbd_local:YS-SK6812MINI-E -> kbd:YS-SK6812MINI-E
- LED47: renamed from LED5; footprint kbd_local:YS-SK6812MINI-E -> kbd:YS-SK6812MINI-E
- LED48: renamed from LED6; footprint kbd_local:YS-SK6812MINI-E -> kbd:YS-SK6812MINI-E
- LED49: renamed from LED7; footprint kbd_local:YS-SK6812MINI-E -> kbd:YS-SK6812MINI-E
- LED50: renamed from LED8; footprint kbd_local:YS-SK6812MINI-E -> kbd:YS-SK6812MINI-E
- LED51: renamed from LED4; footprint kbd_local:YS-SK6812MINI-E -> kbd:YS-SK6812MINI-E
- LED52: renamed from LED3; footprint kbd_local:YS-SK6812MINI-E -> kbd:YS-SK6812MINI-E
- LED53: renamed from LED2; footprint kbd_local:YS-SK6812MINI-E -> kbd:YS-SK6812MINI-E
- LED54: renamed from LED1; footprint kbd_local:YS-SK6812MINI-E -> kbd:YS-SK6812MINI-E
- renumbered C1 to C17, C2 to C18, C3 to C19, C4 to C20, C5 to C21, C6 to C22, C7 to C23, C8 to C24, C9 to C25, C10 to C26, C11 to C27, C12 to C28, C13 to C29, C14 to C30, C15 to C31, C16 to C32, D1 to D49, J4 to J10, JP1 to JP2, R1 to R10, R2 to R11, R3 to R12, R4 to R13, R5 to R14, R8 to R15, R9 to R16, R6 to R17, R7 to R18, SMDSW2 to SMDSW3, SMDSW1 to SMDSW4, SW19 to SW24, SW20 to SW25, SW21 to SW26, SW18 to SW27, SW17 to SW28, SW16 to SW29, SW13 to SW30, SW14 to SW31, SW15 to SW32, SW12 to SW33, SW11 to SW34, SW10 to SW35, SW9 to SW36, SW5 to SW37, SW6 to SW38, SW7 to SW39, SW8 to SW40, SW4 to SW41, SW3 to SW42, SW2 to SW43, SW1 to SW44, U1 to U6, U2 to U7, U3 to U8, U4 to U9, Y1 to Y2, ZD1 to ZD2
