File: Plates/contra-plate/contra-plate.kicad_pcb (KiCad board)
At the start: 2 copper layers, 251.5 x 76.2 mm, 0 parts

Commit message: move switch cutouts to edge.cuts layer
Other:
- outline, holes or cut-outs redrawn
- board text added: "Contra+ by ReillyBex"
