File: contra-plate/contra-plate.kicad_pcb (KiCad board)
At the start: 2 copper layers, 251.5 x 76.2 mm, 0 parts

Commit message: update plate pcb to have gasket pads
Other:
- board size 251.5 x 76.2 mm -> 251.5 x 83.8 mm
- board text added: "Dumortierite by ReillyBex"
- board text removed: "Contra+ by ReillyBex"
