File: PCB/Contra.kicad_pcb (KiCad board)
At the start: 2 copper layers, 251.5 x 76.2 mm, 152 parts, among them J1 Conn_01x03, J2 Conn_01x02, SW1 SW_PUSH, SW2 SW_SPDT, U1 ProMicro

Commit message: update to use local footprints
Parts:
- K1: renamed from MX1; value MX-1U -> KEYSW; footprint MX_Hotswap:MX-Hotswap-1U -> Local-lib:MX-Hotswap-1U
- K10: renamed from MX10; value MX-1U -> KEYSW; footprint MX_Hotswap:MX-Hotswap-1U -> Local-lib:MX-Hotswap-1U
- K11: renamed from MX11; value MX-1U -> KEYSW; footprint MX_Hotswap:MX-Hotswap-1U -> Local-lib:MX-Hotswap-1U
- K12: renamed from MX12; value MX-1U -> KEYSW; footprint MX_Hotswap:MX-Hotswap-1U -> Local-lib:MX-Hotswap-1U
- K13: renamed from MX13; value MX-1U -> KEYSW; footprint MX_Hotswap:MX-Hotswap-1U -> Local-lib:MX-Hotswap-1U
- K14: renamed from MX14; value MX-1U -> KEYSW; footprint MX_Hotswap:MX-Hotswap-1U -> Local-lib:MX-Hotswap-1U
- K15: renamed from MX15; value MX-1U -> KEYSW; footprint MX_Hotswap:MX-Hotswap-1U -> Local-lib:MX-Hotswap-1U
- K16: renamed from MX16; value MX-1U -> KEYSW; footprint MX_Hotswap:MX-Hotswap-1U -> Local-lib:MX-Hotswap-1U
- K17: renamed from MX17; value MX-1U -> KEYSW; footprint MX_Hotswap:MX-Hotswap-1U -> Local-lib:MX-Hotswap-1U
- K18: renamed from MX18; value MX-1U -> KEYSW; footprint MX_Hotswap:MX-Hotswap-1U -> Local-lib:MX-Hotswap-1U
- K19: renamed from MX19; value MX-1U -> KEYSW; footprint MX_Hotswap:MX-Hotswap-1U -> Local-lib:MX-Hotswap-1U
- K2: renamed from MX2; value MX-1U -> KEYSW; footprint MX_Hotswap:MX-Hotswap-1U -> Local-lib:MX-Hotswap-1U
- K20: renamed from MX20; value MX-1U -> KEYSW; footprint MX_Hotswap:MX-Hotswap-1U -> Local-lib:MX-Hotswap-1U
- K21: renamed from MX21; value MX-1U -> KEYSW; footprint MX_Hotswap:MX-Hotswap-1U -> Local-lib:MX-Hotswap-1U
- K22: renamed from MX22; value MX-1U -> KEYSW; footprint MX_Hotswap:MX-Hotswap-1U -> Local-lib:MX-Hotswap-1U
- K23: renamed from MX23; value MX-1U -> KEYSW; footprint MX_Hotswap:MX-Hotswap-1U -> Local-lib:MX-Hotswap-1U
- K24: renamed from MX24; value MX-1U -> KEYSW; footprint MX_Hotswap:MX-Hotswap-1U -> Local-lib:MX-Hotswap-1U
- K25: renamed from MX25; value MX-1U -> KEYSW; footprint MX_Hotswap:MX-Hotswap-1U -> Local-lib:MX-Hotswap-1U
- K26: renamed from MX26; value MX-1U -> KEYSW; footprint MX_Hotswap:MX-Hotswap-1U -> Local-lib:MX-Hotswap-1U
- K27: renamed from MX27; value MX-1U -> KEYSW; footprint MX_Hotswap:MX-Hotswap-1U -> Local-lib:MX-Hotswap-1U
- K28: renamed from MX28; value MX-1U -> KEYSW; footprint MX_Hotswap:MX-Hotswap-1U -> Local-lib:MX-Hotswap-1U
- K29: renamed from MX29; value MX-1U -> KEYSW; footprint MX_Hotswap:MX-Hotswap-1U -> Local-lib:MX-Hotswap-1U
- K3: renamed from MX3; value MX-1U -> KEYSW; footprint MX_Hotswap:MX-Hotswap-1U -> Local-lib:MX-Hotswap-1U
- K30: renamed from MX30; value MX-1U -> KEYSW; footprint MX_Hotswap:MX-Hotswap-1U -> Local-lib:MX-Hotswap-1U
- K31: renamed from MX31; value MX-1U -> KEYSW; footprint MX_Hotswap:MX-Hotswap-1U -> Local-lib:MX-Hotswap-1U
- K32: renamed from MX32; value MX-1U -> KEYSW; footprint MX_Hotswap:MX-Hotswap-1U -> Local-lib:MX-Hotswap-1U
- K33: renamed from MX33; value MX-1U -> KEYSW; footprint MX_Hotswap:MX-Hotswap-1U -> Local-lib:MX-Hotswap-1U
- K34: renamed from MX34; value MX-1U -> KEYSW; footprint MX_Hotswap:MX-Hotswap-1U -> Local-lib:MX-Hotswap-1U
- K35: renamed from MX35; value MX-1U -> KEYSW; footprint MX_Hotswap:MX-Hotswap-1U -> Local-lib:MX-Hotswap-1U
- K36: renamed from MX36; value MX-1U -> KEYSW; footprint MX_Hotswap:MX-Hotswap-1U -> Local-lib:MX-Hotswap-1U
- K37: renamed from MX37; value MX-1U -> KEYSW; footprint MX_Hotswap:MX-Hotswap-1U -> Local-lib:MX-Hotswap-1U
- K38: renamed from MX38; value MX-1U -> KEYSW; footprint MX_Hotswap:MX-Hotswap-1U -> Local-lib:MX-Hotswap-1U
- K39: renamed from MX39; value MX-1U -> KEYSW; footprint MX_Hotswap:MX-Hotswap-1U -> Local-lib:MX-Hotswap-1U
- K4: renamed from MX4; value MX-1U -> KEYSW; footprint MX_Hotswap:MX-Hotswap-1U -> Local-lib:MX-Hotswap-1U
- K40: renamed from MX40; value MX-1U -> KEYSW; footprint MX_Hotswap:MX-Hotswap-1U -> Local-lib:MX-Hotswap-1U
- K41: renamed from MX41; value MX-1U -> KEYSW; footprint MX_Hotswap:MX-Hotswap-1U -> Local-lib:MX-Hotswap-1U
- K42: renamed from MX42; value MX-2U -> KEYSW; footprint MX_Hotswap:MX-Hotswap-2U-ReversedStabilizers -> Local-lib:MX-Hotswap-2U-ReversedStabilizers
- K43: renamed from MX43; value MX-1U -> KEYSW; footprint MX_Hotswap:MX-Hotswap-1U -> Local-lib:MX-Hotswap-1U
- K44: renamed from MX44; value MX-1U -> KEYSW; footprint MX_Hotswap:MX-Hotswap-1U -> Local-lib:MX-Hotswap-1U
- K45: renamed from MX45; value MX-1U -> KEYSW; footprint MX_Hotswap:MX-Hotswap-1U -> Local-lib:MX-Hotswap-1U
- K46: renamed from MX46; value MX-1U -> KEYSW; footprint MX_Hotswap:MX-Hotswap-1U -> Local-lib:MX-Hotswap-1U
- K47: renamed from MX47; value MX-1U -> KEYSW; footprint MX_Hotswap:MX-Hotswap-1U -> Local-lib:MX-Hotswap-1U
- K5: renamed from MX5; value MX-1U -> KEYSW; footprint MX_Hotswap:MX-Hotswap-1U -> Local-lib:MX-Hotswap-1U
- K6: renamed from MX6; value MX-1U -> KEYSW; footprint MX_Hotswap:MX-Hotswap-1U -> Local-lib:MX-Hotswap-1U
- K7: renamed from MX7; value MX-1U -> KEYSW; footprint MX_Hotswap:MX-Hotswap-1U -> Local-lib:MX-Hotswap-1U
- K8: renamed from MX8; value MX-1U -> KEYSW; footprint MX_Hotswap:MX-Hotswap-1U -> Local-lib:MX-Hotswap-1U
- K9: renamed from MX9; value MX-1U -> KEYSW; footprint MX_Hotswap:MX-Hotswap-1U -> Local-lib:MX-Hotswap-1U
- LED1, LED10, LED11, LED12, LED13, LED14, LED15, LED16, LED17, LED18, LED19, LED2, LED20, LED21, LED22, LED23, LED24, LED25, LED26, LED27, LED28, LED29, LED3, LED30, LED31, LED32, LED33, LED34, LED35, LED36, LED37, LED38, LED39, LED4, LED40, LED41, LED42, LED43, LED44, LED45, LED46, LED47, LED5, LED6, LED7, LED8, LED9: value 4960 -> SK6812-ReverseMount; footprint kbd:YS-SK6812MINI-E -> Local-lib:YS-SK6812MINI-E
- OL1: footprint kbd:OLED -> Local-lib:OLED
- U1: value ProMicro -> SuperMini nRF52840; footprint Reilly_Components:SuperMini NRF52840 -> Local-lib:SuperMini NRF52840

Commit message: add silkscreen name to pcb
Other:
- board text added: "Dumortierite by ReillyBex"
Changed lines of the file:
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@@
 		(tags "mountinghole M2")
 		(property "Reference" "H2"
-			(at 0 -3.15 0)
+			(at 0.0575 3.39 0)
 			(layer "F.SilkS")
 			(effects
@@
 		)
 	)
+	(gr_text "Dumortierite\nby\nReillyBex"
+		(at 34.29 118.11 0)
+		(layer "B.SilkS")
+		(effects
+			(font
+				(size 1.5 1.5)
+				(thickness 0.3)
+				(bold yes)
+			)
+			(justify bottom mirror)
+		)
+	)

Commit message: update 1u footprints adjust spacing
Parts:
- removed H1: MountingHole, MountingHole:MountingHole_2.2mm_M2
- removed H2, H3, H4, H5: MountingHole_Pad, MountingHole:MountingHole_2.2mm_M2_Pad
- K1, K10, K11, K12, K13, K14, K15, K16, K17, K18, K19, K2, K20, K21, K22, K23, K24, K25, K26, K27, K28, K29, K3, K30, K31, K32, K33, K34, K35, K36, K37, K38, K39, K4, K40, K41, K43, K44, K45, K46, K47, K5, K6, K7, K8, K9: footprint Local-lib:MX-Hotswap-1U -> Local-lib:keyswitch_choc12_hotswap_1u
- moved D1 0.95 mm to (63.5, 61.9)
- moved D10 0.95 mm to (234.9, 61.9)
- moved D11 0.95 mm to (254.0, 61.9)
- moved D12 0.95 mm to (273.1, 61.9)
- moved D13 0.95 mm to (63.5, 81.0)
- moved D14 0.95 mm to (82.5, 81.0)
- moved D15 0.95 mm to (101.6, 81.0)
- moved D16 0.95 mm to (120.7, 81.0)
- moved D17 0.95 mm to (139.7, 81.0)
- moved D18 0.95 mm to (158.8, 81.0)
- moved D19 0.95 mm to (177.8, 81.0)
- moved D2 0.95 mm to (82.5, 61.9)
- moved D20 0.95 mm to (196.8, 81.0)
- moved D21 0.95 mm to (215.9, 81.0)
- moved D22 0.95 mm to (234.9, 81.0)
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Routing:
- net ROW0: track 225.8 -> 254.5 mm
- net ROW2: track 242.2 -> 270.7 mm
- net ROW1: track 228.3 -> 255.8 mm
- net ROW3: track 263.8 -> 288.5 mm
- net COL11: track 349.6 -> 367.0 mm
- net COL2: track 137.9 -> 151.8 mm
- net COL3: track 161.6 -> 175.4 mm
- net COL5: track 185.7 -> 199.1 mm
- net COL10: track 274.3 -> 287.5 mm
- net COL9: track 255.8 -> 268.4 mm
- net COL4: track 162.4 -> 174.8 mm
- net COL8: track 236.5 -> 248.7 mm
- net COL1: track 116.7 -> 128.6 mm
- net COL7: track 216.9 -> 228.5 mm
- net COL6: track 178.0 -> 186.6 mm
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